File: electronics/SmartScale.kicad_sch (KiCad schematic)
At the start: 66 parts, among them IC1 HX711, IC2 632723100011, J2 Conn_01x06, J3 Conn_01x06, J4 Conn_01x04, Q1 BC847, Q2 BC847, Q3 IRLML0030, Q4 IRLML0030, Q5 MMBT3906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

Commit message: PCB Rev 6, fixed error with flashing
Connections:
- net DTR: now also Q1.2 (E)
- net RTS: now also Q2.2 (E)
- net at Q1.1 (B), R1.1: no longer Q2.2 (E)
- net at Q2.1 (B), R2.1: no longer Q1.2 (E)
Other:
- note added: "USB-C"
- moved on the sheet: Q1, Q2, R1, R2

Commit message: Intermediate push, dunno what I just broke but whatever
Other:
- note added: "Alternativen: IRLML 0100"
- note added: "LiPo Protection"
Changed lines of the file:
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@@
     (stroke (width 0) (type default) (color 0 0 0 0))
   )
-  (text "TP Lademodul" (at 154.94 139.7 0)
+  (text "Alternativen:\nIRLML 0100" (at 203.2 143.51 0)
+    (effects (font (size 1.27 1.27)) (justify left bottom))
+  )
+  (text "TP Lademodul" (at 96.52 143.51 0)
     (effects (font (size 1.27 1.27)) (justify left bottom))
   )
@@
     (effects (font (size 1.27 1.27)) (justify left bottom))
   )
+  (text "LiPo Protection" (at 154.94 113.03 0)
+    (effects (font (size 1.27 1.27)) (justify left bottom))
+  )

Commit message: Push after a long time
Other:
- note added: "MOSFET Ron = 0,15V / 2*MaxAmp 3.80A -> 20mOhm 1.90A -> 40mOhm 1.00A -> 75mOhm 0.80A -> 100mOhm 0.50A -> 150mOhm 0.38A -> 200mOhm 0.30A -> 250mOhm 0.25A -> 300mOhm"
- note added: "Overcurrent on CS Pin: 0.15V and 1.35V MaxAmp = 0.15V / (2 * Ron)"
- note removed: "MOSFET Ron = 0,15V / 2*MaxAmp 1.0A -> 75mOhm 0.8A -> 100mOhm 0.5A -> 150mOhm 0.3A -> 250mOhm"
Changed lines of the file:
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@@
     (stroke (width 0) (type default) (color 0 0 0 0))
   )
-  (wire (pts (xy 147.32 121.92) (xy 147.32 148.59))
+  (wire (pts (xy 146.05 121.92) (xy 146.05 148.59))
     (stroke (width 0) (type default) (color 0 0 0 0))
   )
@@
     (stroke (width 0) (type default) (color 0 0 0 0))
   )
+  (wire (pts (xy 209.55 95.25) (xy 209.55 96.52))
+    (stroke (width 0) (type default) (color 0 0 0 0))
+  )
   (wire (pts (xy 227.33 73.66) (xy 227.33 53.34))
     (stroke (width 0) (type default) (color 0 0 0 0))
@@
     (stroke (width 0) (type default) (color 0 0 0 0))
   )
-  (wire (pts (xy 147.32 148.59) (xy 185.42 148.59))
+  (wire (pts (xy 146.05 148.59) (xy 185.42 148.59))
     (stroke (width 0) (type default) (color 0 0 0 0))
   )
@@
     (stroke (width 0) (type default) (color 0 0 0 0))
   )
+  (wire (pts (xy 173.99 139.7) (xy 173.99 138.43))
+    (stroke (width 0) (type default) (color 0 0 0 0))
+  )
   (wire (pts (xy 227.33 35.56) (xy 227.33 27.94))
     (stroke (width 0) (type default) (color 0 0 0 0))
@@
     (stroke (width 0) (type default) (color 0 0 0 0))
   )
-  (wire (pts (xy 156.21 121.92) (xy 147.32 121.92))
+  (wire (pts (xy 156.21 121.92) (xy 146.05 121.92))
     (stroke (width 0) (type default) (color 0 0 0 0))
   )
@@
   (text "TP Lademodul" (at 96.52 143.51 0)
     (effects (font (size 1.27 1.27)) (justify left bottom))
+  )
+  (text "Overcurrent on CS Pin:\n0.15V and 1.35V\nMaxAmp = 0.15V / (2 * Ron)"
+    (at 184.15 158.75 0)
+    (effects (font (size 1 1)) (justify left bottom))
   )
   (text "USB-C" (at 53.34 172.72 0)
@@
     (effects (font (size 1.27 1.27)) (justify left bottom))
   )
-  (text "MOSFET Ron = 0,15V / 2*MaxAmp\n1.0A -> 75mOhm \n0.8A -> 100mOhm\n0.5A -> 150mOhm\n0.3A -> 250mOhm"
-    (at 162.56 162.56 0)
-    (effects (font (size 1.27 1.27)) (justify left bottom))
+  (text "MOSFET Ron = 0,15V / 2*MaxAmp\n3.80A ->  20mOhm\n1.90A ->  40mOhm\n1.00A ->  75mOhm\n0.80A -> 100mOhm\n0.50A -> 150mOhm\n0.38A -> 200mOhm\n0.30A -> 250mOhm\n0.25A -> 300mOhm"
+    (at 154.94 167.64 0)
+    (effects (font (size 1 1)) (justify left bottom))
   )
   (text "Input: > 1uF\nOutput: > 10uF" (at 250.19 123.19 0)
@@
     (effects (font (size 1.27 1.27)) (justify left bottom))
   )
-  (text "130mA\n250mA\n300mA\n400mA\n580mA\n690mA\n780mA\n900mA\n1000mA"
+  (text " 130mA\n 250mA\n 300mA\n 400mA\n 580mA\n 690mA\n 780mA\n 900mA\n1000mA"
     (at 135.89 193.04 0)
     (effects (font (size 1.27 1.27)) (justify left bottom))
@@
     (pin "3")
   )
-  (symbol (lib_id "SmartScale-rescue:GND-power") (at 173.99 138.43 0) (unit 1)
-    (in_bom yes) (on_board yes)
-    (property "Reference" "#PWR021" (id 0) (at 173.99 144.78 0)
-      (effects (font (size 1.27 1.27)) hide)
-    )
-    (property "Value" "GND" (id 1) (at 174.117 142.8242 0))
-    (property "Footprint" "" (id 2) (at 173.99 138.43 0)
-      (effects (font (size 1.27 1.27)) hide)
-    )
-    (property "Datasheet" "" (id 3) (at 173.99 138.43 0)
+  (symbol (lib_id "SmartScale-rescue:GND-power") (at 173.99 139.7 0) (unit 1)
+    (in_bom yes) (on_board yes)
+    (property "Reference" "#PWR021" (id 0) (at 173.99 146.05 0)
+      (effects (font (size 1.27 1.27)) hide)
+    )
+    (property "Value" "GND" (id 1) (at 174.117 144.0942 0))
+    (property "Footprint" "" (id 2) (at 173.99 139.7 0)
+      (effects (font (size 1.27 1.27)) hide)
+    )
+    (property "Datasheet" "" (id 3) (at 173.99 139.7 0)
       (effects (font (size 1.27 1.27)) hide)
     )
@@
     (pin "2")
   )
-  (symbol (lib_id "power:GND") (at 209.55 96.52 180) (unit 1)
-    (in_bom yes) (on_board yes)
-    (property "Reference" "#PWR024" (id 0) (at 209.55 90.17 0)
-      (effects (font (size 1.27 1.27)) hide)
-    )
-    (property "Value" "GND" (id 1) (at 209.423 92.1258 0))
-    (property "Footprint" "" (id 2) (at 209.55 96.52 0)
-      (effects (font (size 1.27 1.27)) hide)
-    )
-    (property "Datasheet" "" (id 3) (at 209.55 96.52 0)
-      (effects (font (size 1.27 1.27)) hide)
-    )
+  (symbol (lib_id "power:GND") (at 209.55 95.25 180) (unit 1)
+    (in_bom yes) (on_board yes)
+    (property "Reference" "#PWR024" (id 0) (at 209.55 88.9 0)
+      (effects (font (size 1.27 1.27)) hide)
+    )
+    (property "Value" "GND" (id 1) (at 209.423 90.8558 0))
+    (property "Footprint" "" (id 2) (at 209.55 95.25 0)
+      (effects (font (size 1.27 1.27)) hide)
+    )
+    (property "Datasheet" "" (id 3) (at 209.55 95.25 0)
+      (effects (font (size 1.27 1.27)) hide)
+    )
